File: top.kicad_pcb (KiCad board)
At the start: 2 copper layers, 85 parts, among them IC1 REG113NA-2.5_3K, IC2 LD39015M10R, J1 Conn_01x01_Male, J2 Conn_01x07_Male, SW1 SW_SPDT, U1 digital clock, U2 BC2AAPC, Y1 Crystal 32.768kHz

Commit message: Placement done
Parts:
- D2, D3, D4, D5: footprint top_footprintlib:SOT95P280X145-5N -> LED_SMD:LED_0603_1608Metric_Pad1.05x0.95mm_HandSolder
- moved S4 158.5 mm to (170.2, 173.4)
- moved S2 143.0 mm to (137.2, 173.4)
- moved C8 142.8 mm to (168.9, 90.8)
- moved R7 140.6 mm to (151.1, 161.9), turned to -90 degrees
- moved S1 138.4 mm to (120.7, 173.4)
- moved C4 138.0 mm to (177.8, 161.9), turned to -90 degrees
- moved C5 133.8 mm to (106.7, 161.9), turned to 90 degrees
- moved S3 133.7 mm to (153.7, 173.4)
- moved R8 129.9 mm to (167.6, 161.9), turned to -90 degrees
- moved R12 129.7 mm to (172.7, 161.9), turned to 90 degrees
- moved C7 129.1 mm to (161.3, 87.0), turned to 180 degrees
- moved D3 129.0 mm to (132.5, 152.1), turned to -90 degrees
- moved C2 125.4 mm to (144.8, 161.9), turned to -90 degrees
- moved D5 123.1 mm to (143.7, 152.1), turned to -90 degrees
- moved C3 122.0 mm to (161.3, 161.9), turned to -90 degrees
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Routing:
- net RESETN: track 0.00 -> 106.2 mm
- net DIGIT_3: track 0.00 -> 39.2 mm
- net Net-(DS1-Pad11): track 0.00 -> 38.5 mm, vias 0 -> 1
- net Net-(DS1-Pad15): track 0.00 -> 37.7 mm, vias 0 -> 1
- net Net-(DS1-Pad12): track 0.00 -> 36.6 mm
- net DIGIT_4: track 0.00 -> 35.4 mm
- net Net-(DS1-Pad6): track 0.00 -> 31.4 mm
- net Net-(DS1-Pad4): track 0.00 -> 20.3 mm, vias 0 -> 1
- net G: track 0.00 -> 19.8 mm
- net Net-(R12-Pad1): track 0.00 -> 19.6 mm
- net Net-(R11-Pad1): track 0.00 -> 19.6 mm
- net Net-(R5-Pad2): track 0.00 -> 19.6 mm
- net Net-(R10-Pad1): track 0.00 -> 19.6 mm
- net DP: track 0.00 -> 19.2 mm
- net E: track 0.00 -> 16.7 mm
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
Commit message: Final
Parts:
- moved S3 141.2 mm to (117.6, 36.8), turned to 90 degrees
- moved S4 138.8 mm to (145.2, 36.8), turned to 90 degrees
- moved S1 137.7 mm to (102.7, 36.8), turned to 90 degrees
- moved S5 137.6 mm to (88.1, 36.6), turned to 90 degrees
- moved S2 136.6 mm to (131.4, 36.8), turned to 90 degrees
- moved C4 126.5 mm to (123.4, 47.7), turned to 90 degrees
- moved C3 125.8 mm to (108.6, 47.7), turned to 90 degrees
- moved R12 123.0 mm to (127.1, 47.8), turned to -90 degrees
- moved R11 122.4 mm to (112.2, 47.8), turned to -90 degrees
- moved R8 120.0 mm to (130.7, 47.8), turned to 90 degrees
- moved C1 118.6 mm to (96.1, 47.7), turned to 90 degrees
- moved C2 117.8 mm to (115.9, 47.7), turned to 90 degrees
- moved R10 115.9 mm to (119.8, 47.8), turned to -90 degrees
- moved R9 115.8 mm to (103.8, 47.8), turned to -90 degrees
- moved C5 115.7 mm to (88.4, 47.7)
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Connections:
- SW1 pad 4: (no net) -> GND
- SW1 pad 5: (no net) -> GND
Routing:
- net +1V0: track 0.00 -> 234.7 mm, vias 0 -> 2
- net GND: track 0.00 -> 227.6 mm, vias 0 -> 3
- net DIGIT_5: track 0.00 -> 105.3 mm, vias 0 -> 1
- net +2V5: track 0.00 -> 95.3 mm
- net Net-(DS1-Pad2): track 0.00 -> 74.1 mm
- net Net-(SW1-Pad3): track 0.00 -> 61.7 mm
- net Net-(DS1-Pad3): track 0.00 -> 60.5 mm
- net RESETN: track 106.2 -> 48.1 mm
- net DIGIT_2: track 0.00 -> 56.1 mm
- net DIGIT_1: track 0.00 -> 54.6 mm
- net EXTERNAL_1HZ_ENABLE: track 0.00 -> 53.5 mm
- net BUZZER: track 0.00 -> 51.4 mm
- net DIGIT_3: track 39.2 -> 85.4 mm
- net ONE_HZ_TEST: track 0.00 -> 45.4 mm
- net +3V0: track 0.00 -> 44.8 mm
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- added copper zone on B.Cu, net GND
- added copper zone on F.Cu, net GND
Other:
- board outline added: 132.7 x 146.9 mm
- board text added: "0"
- board text added: "1"
- board text added: "1HZ TEST"
- board text added: "1V Switch"
- board text added: "2"
- board text added: "2.5V Switch"
- board text added: "3"
- board text added: "4"
- board text added: "5"
- board text added: "6"
- board text added: "ADV CLK EN"
- board text added: "ADV HOUR"
- board text added: "ADV MIN"
- board text added: "Alarm"
- board text added: "Clock"
- board text added: "Digit Switch"
- board text added: "EE 6350 Digital Clock Columbia University Fall 2022"
- board text added: "EXT 1HZ EN"
- board text added: "EXT 1HZ IN"
- board text added: "EXT CLK"
- board text added: "EXT CLK EN"
- board text added: "Modes"
- board text added: "POWER ON<->OFF"
- board text added: "Reset"
- board text added: "SEG_BAR TEST PIN"
- board text added: "Set Time"
- board text added: "Start"
- board text added: "Switch Mode"
- board text added: "TEST MUX 3-1 0"
- board text added: "TEST MUX 3-1 1"
- board text added: "TEST MUX 6-1 0"
- board text added: "TEST MUX 6-1 1"
- board text added: "TEST MUX 6-1 2"
- board text added: "TEST MUX EN"
- board text added: "Time Plus"
- board text added: "Timer"
- board text added: "XIN"
- board text added: "XOUT"
- board text added: "h h : m m : s s"
