File: top.kicad_sch (KiCad schematic)
At the start: 84 parts, among them IC1 REG113NA-2.5_3K, IC2 LD39015M10R, J1 Conn_01x01_Male, J2 Conn_01x07_Male, U1 digital clock, U2 BC2AAPC, Y1 Crystal 32.768kHz

Commit message: Placement done
Parts:
- added SW1: SW_SPDT, symbol Switch:SW_SPDT
- D2, D3, D4, D5: footprint top_footprintlib:SOT95P280X145-5N -> LED_SMD:LED_0603_1608Metric_Pad1.05x0.95mm_HandSolder
Connections:
- net +3V0: now also SW1.2 (B); no longer U2.1 (+)
- new net: SW1.3 (C), U2.1 (+)
Changed lines of the file:
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@@
     (stroke (width 0) (type default) (color 0 0 0 0))
   )
+  (wire (pts (xy 335.28 32.385) (xy 335.28 27.305))
+    (stroke (width 0) (type default) (color 0 0 0 0))
+  )
   (wire (pts (xy 242.57 21.59) (xy 242.57 22.86))
     (stroke (width 0) (type default) (color 0 0 0 0))
@@
     (stroke (width 0) (type default) (color 0 0 0 0))
   )
-  (wire (pts (xy 334.645 27.305) (xy 332.74 27.305))
+  (wire (pts (xy 332.74 27.305) (xy 335.28 27.305))
     (stroke (width 0) (type default) (color 0 0 0 0))
   )
@@
     (stroke (width 0) (type default) (color 0 0 0 0))
   )
-  (wire (pts (xy 334.645 22.225) (xy 334.645 27.305))
-    (stroke (width 0) (type default) (color 0 0 0 0))
-  )
   (polyline (pts (xy 12.065 68.58) (xy 64.77 68.58))
     (stroke (width 0) (type default) (color 0 0 0 0))
@@
     (stroke (width 0) (type default) (color 0 0 0 0))
   )
+  (wire (pts (xy 345.44 34.925) (xy 347.98 34.925))
+    (stroke (width 0) (type default) (color 0 0 0 0))
+  )
   (wire (pts (xy 55.245 171.45) (xy 55.245 175.26))
     (stroke (width 0) (type default) (color 0 0 0 0))
@@
     (property "Reference" "D3" (id 0) (at 33.02 43.815 0))
     (property "Value" "LED" (id 1) (at 33.02 46.355 0))
-    (property "Footprint" "top_footprintlib:SOT95P280X145-5N" (id 2) (at 24.765 49.53 0)
+    (property "Footprint" "LED_SMD:LED_0603_1608Metric_Pad1.05x0.95mm_HandSolder" (id 2) (at 24.765 49.53 0)
       (effects (font (size 1.27 1.27)) hide)
     )
@@
     (pin "1")
   )
+  (symbol (lib_id "power:+3V0") (at 347.98 34.925 0) (unit 1)
+    (in_bom yes) (on_board yes) (fields_autoplaced)
+    (property "Reference" "#PWR?" (id 0) (at 347.98 38.735 0)
+      (effects (font (size 1.27 1.27)) hide)
+    )
+    (property "Value" "+3V0" (id 1) (at 347.98 29.21 0))
+    (property "Footprint" "" (id 2) (at 347.98 34.925 0)
+      (effects (font (size 1.27 1.27)) hide)
+    )
+    (property "Datasheet" "" (id 3) (at 347.98 34.925 0)
+      (effects (font (size 1.27 1.27)) hide)
+    )
+    (pin "1")
+  )
   (symbol (lib_id "Jumper:Jumper_3_Bridged12") (at 256.54 22.86 0) (unit 1)
     (in_bom yes) (on_board yes) (fields_autoplaced)
@@
     (property "Reference" "D5" (id 0) (at 33.02 57.15 0))
     (property "Value" "LED" (id 1) (at 33.02 59.69 0))
-    (property "Footprint" "top_footprintlib:SOT95P280X145-5N" (id 2) (at 24.765 62.865 0)
+    (property "Footprint" "LED_SMD:LED_0603_1608Metric_Pad1.05x0.95mm_HandSolder" (id 2) (at 24.765 62.865 0)
       (effects (font (size 1.27 1.27)) hide)
     )
@@
     (pin "1")
   )
+  (symbol (lib_id "Switch:SW_SPDT") (at 340.36 34.925 180) (unit 1)
+    (in_bom yes) (on_board yes) (fields_autoplaced)
+    (property "Reference" "SW1" (id 0) (at 340.36 26.67 0))
+    (property "Value" "SW_SPDT" (id 1) (at 340.36 29.21 0))
+    (property "Footprint" "" (id 2) (at 340.36 34.925 0)
+      (effects (font (size 1.27 1.27)) hide)
+    )
+    (property "Datasheet" "~" (id 3) (at 340.36 34.925 0)
+      (effects (font (size 1.27 1.27)) hide)
+    )
+    (pin "1")
+    (pin "2")
+    (pin "3")
+  )
   (symbol (lib_id "Device:R") (at 184.15 252.73 0) (unit 1)
     (in_bom yes) (on_board yes) (fields_autoplaced)
@@
     (property "Reference" "D2" (id 0) (at 33.02 37.465 0))
     (property "Value" "LED" (id 1) (at 33.02 40.005 0))
-    (property "Footprint" "top_footprintlib:SOT95P280X145-5N" (id 2) (at 24.765 43.18 0)
+    (property "Footprint" "LED_SMD:LED_0603_1608Metric_Pad1.05x0.95mm_HandSolder" (id 2) (at 24.765 43.18 0)
       (effects (font (size 1.27 1.27)) hide)
     )
@@
     (pin "3")
   )
-  (symbol (lib_id "power:+3V0") (at 334.645 22.225 0) (unit 1)
-    (in_bom yes) (on_board yes) (fields_autoplaced)
-    (property "Reference" "#PWR044" (id 0) (at 334.645 26.035 0)
-      (effects (font (size 1.27 1.27)) hide)
-    )
-    (property "Value" "+3V0" (id 1) (at 334.645 16.51 0))
-    (property "Footprint" "" (id 2) (at 334.645 22.225 0)
-      (effects (font (size 1.27 1.27)) hide)
-    )
-    (property "Datasheet" "" (id 3) (at 334.645 22.225 0)
-      (effects (font (size 1.27 1.27)) hide)
-    )
-    (pin "1")
-  )
   (symbol (lib_id "Device:C") (at 76.835 182.88 0) (unit 1)
     (in_bom yes) (on_board yes) (fields_autoplaced)
@@
     (property "Reference" "D4" (id 0) (at 33.02 50.8 0))
     (property "Value" "LED" (id 1) (at 33.02 53.34 0))
-    (property "Footprint" "top_footprintlib:SOT95P280X145-5N" (id 2) (at 24.765 56.515 0)
+    (property "Footprint" "LED_SMD:LED_0603_1608Metric_Pad1.05x0.95mm_HandSolder" (id 2) (at 24.765 56.515 0)
       (effects (font (size 1.27 1.27)) hide)
     )
@@
       (reference "#PWR043") (unit 1) (value "GND") (footprint "")
     )
-    (path "/db10b2fa-ef93-481a-a1cc-7b0c34f5aedc"
-      (reference "#PWR044") (unit 1) (value "+3V0") (footprint "")
-    )
     (path "/1bb098cc-6d84-4604-bdce-97f7c1222283"
       (reference "#PWR045") (unit 1) (value "GND") (footprint "")
@@
       (reference "#PWR061") (unit 1) (value "GND") (footprint "")
     )
+    (path "/402d73c5-d92e-49ae-b268-6dda89905af5"
+      (reference "#PWR?") (unit 1) (value "+3V0") (footprint "")
+    )
     (path "/9fe7834a-8684-4d58-8957-243825e4fdf3"
       (reference "C1") (unit 1) (value "33n") (footprint "Capacitor_SMD:C_1206_3216Metric_Pad1.33x1.80mm_HandSolder")
@@
     )
     (path "/d50c1928-f538-435d-bb3a-5051dcf85e19"
-      (reference "D2") (unit 1) (value "LED") (footprint "top_footprintlib:SOT95P280X145-5N")
+      (reference "D2") (unit 1) (value "LED") (footprint "LED_SMD:LED_0603_1608Metric_Pad1.05x0.95mm_HandSolder")
     )
     (path "/2f8c7f31-8243-4702-8a2a-8ffbf486bc3d"
-      (reference "D3") (unit 1) (value "LED") (footprint "top_footprintlib:SOT95P280X145-5N")
+      (reference "D3") (unit 1) (value "LED") (footprint "LED_SMD:LED_0603_1608Metric_Pad1.05x0.95mm_HandSolder")
     )
     (path "/ecaf978b-fbc1-4b4e-86dc-fd3e1b0e06f8"
-      (reference "D4") (unit 1) (value "LED") (footprint "top_footprintlib:SOT95P280X145-5N")
+      (reference "D4") (unit 1) (value "LED") (footprint "LED_SMD:LED_0603_1608Metric_Pad1.05x0.95mm_HandSolder")
     )
     (path "/7c03227d-5b17-441a-b351-8b8a4841e285"
-      (reference "D5") (unit 1) (value "LED") (footprint "top_footprintlib:SOT95P280X145-5N")
+      (reference "D5") (unit 1) (value "LED") (footprint "LED_SMD:LED_0603_1608Metric_Pad1.05x0.95mm_HandSolder")
     )
     (path "/940ab9a3-160f-447a-b1ac-174a03954a05"
@@
       (reference "S5") (unit 1) (value "HP0315AFKP2-R") (footprint "top_footprintlib:HP0315AFKP2R")
     )
+    (path "/8ebc0ded-a641-4997-90f5-2e7096976fcc"
+      (reference "SW1") (unit 1) (value "SW_SPDT") (footprint "")
+    )
     (path "/5d3d4e6f-52c6-4347-abf7-cf5d4d10f099"

Commit message: Placement done. Require routing
Parts:
- SW1: footprint (none) -> top_footprintlib:SS-12D07-VG
Changed lines of the file:
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@@
   (symbol (lib_id "power:+3V0") (at 347.98 34.925 0) (unit 1)
     (in_bom yes) (on_board yes) (fields_autoplaced)
-    (property "Reference" "#PWR?" (id 0) (at 347.98 38.735 0)
+    (property "Reference" "#PWR0101" (id 0) (at 347.98 38.735 0)
       (effects (font (size 1.27 1.27)) hide)
     )
@@
     (property "Reference" "SW1" (id 0) (at 340.36 26.67 0))
     (property "Value" "SW_SPDT" (id 1) (at 340.36 29.21 0))
-    (property "Footprint" "" (id 2) (at 340.36 34.925 0)
+    (property "Footprint" "top_footprintlib:SS-12D07-VG" (id 2) (at 340.36 34.925 0)
       (effects (font (size 1.27 1.27)) hide)
     )
@@
     )
     (path "/402d73c5-d92e-49ae-b268-6dda89905af5"
-      (reference "#PWR?") (unit 1) (value "+3V0") (footprint "")
+      (reference "#PWR0101") (unit 1) (value "+3V0") (footprint "")
     )
     (path "/9fe7834a-8684-4d58-8957-243825e4fdf3"
@@
     )
     (path "/8ebc0ded-a641-4997-90f5-2e7096976fcc"
-      (reference "SW1") (unit 1) (value "SW_SPDT") (footprint "")
+      (reference "SW1") (unit 1) (value "SW_SPDT") (footprint "top_footprintlib:SS-12D07-VG")
     )
     (path "/5d3d4e6f-52c6-4347-abf7-cf5d4d10f099"

Commit message: Final
Changed lines of the file:
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@@
+    (effects (font (size 1.27 1.27)) (justify left bottom))
+  )
+  (label "battery+" (at 334.645 35.56 90)
     (effects (font (size 1.27 1.27)) (justify left bottom))
   )
